File: KiCAD/RGB Blaster 8DIN Adapter.kicad_pcb (KiCad board)
At the start: 2 copper layers, 28.6 x 18.9 mm, 6 parts, among them P1 Mini_DIN_9P_PCB, P2 8_pin_mini_DIN

Commit message: Changes on KiCAD project
Parts:
- added JP1: Jumper_2_Open, Jumper:SolderJumper-2_P1.3mm_Open_TrianglePad1.0x1.5mm, B.Cu at (135.1, 105.7)
Changed lines of the file:
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@@
   (paper "USLetter")
   (title_block
+    (title "8laster for RGB Blaster")
+    (date "2023-01-29")
     (rev "1")
+    (company "Jeff Chen")
   )
   (layers
@@
       (net 7 "/Red") (pinfunction "R") (pintype "output"))
   )
+  (footprint "Jumper:SolderJumper-2_P1.3mm_Open_TrianglePad1.0x1.5mm" (layer "B.Cu")
+    (at 135.11 105.72 90)
+    (descr "SMD Solder Jumper, 1x1.5mm Triangular Pads, 0.3mm gap, open")
+    (tags "solder jumper open")
+    (property "Sheetfile" "RGB Blaster 8DIN Adapter.kicad_sch")
+    (property "Sheetname" "")
+    (attr exclude_from_pos_files)
+    (fp_text reference "JP1" (at 0.08 2.47) (layer "B.SilkS")
+      (effects (font (size 1 1) (thickness 0.15)) (justify mirror))
+    )
+    (fp_text value "Jumper_2_Open" (at 0 -1.9 90) (layer "B.Fab")
+      (effects (font (size 1 1) (thickness 0.15)) (justify mirror))
+    )
+    (fp_line (start -1.4 1) (end 1.4 1) (layer "B.SilkS") (width 0.12))
+    (fp_line (start 1.4 -1) (end -1.4 -1) (layer "B.SilkS") (width 0.12))
+    (fp_line (start 1.4 1) (end 1.4 -1) (layer "B.SilkS") (width 0.12))
+    (fp_line (start -1.4 -1) (end -1.4 1) (layer "B.SilkS") (width 0.12))
+    (fp_line (start 1.65 -1.25) (end -1.65 -1.25) (layer "B.CrtYd") (width 0.05))
+    (fp_line (start -1.65 1.25) (end 1.65 1.25) (layer "B.CrtYd") (width 0.05))
+    (fp_line (start 1.65 -1.25) (end 1.65 1.25) (layer "B.CrtYd") (width 0.05))
+    (fp_line (start -1.65 1.25) (end -1.65 -1.25) (layer "B.CrtYd") (width 0.05))
+    (pad "1" smd custom (at -0.725 0 90) (size 0.3 0.3) (layers "B.Cu" "B.Mask")
+      (net 4 "/Sync") (pinfunction "A") (pintype "passive") (zone_connect 2)
+      (options (clearance outline) (anchor rect))
+      (primitives
+        (gr_poly (pts
+            (xy 1 0)
+            (xy 0.5 -0.75)
+            (xy -0.5 -0.75)
+            (xy -0.5 0.75)
+            (xy 0.5 0.75)
+          ) (width 0) (fill yes))
+      ))
+    (pad "2" smd custom (at 0.725 0 90) (size 0.3 0.3) (layers "B.Cu" "B.Mask")
+      (net 11 "/Attenuated Sync") (pinfunction "B") (pintype "passive") (zone_connect 2)
+      (options (clearance outline) (anchor rect))
+      (primitives
+        (gr_poly (pts
+            (xy 0.5 -0.75)
+            (xy -0.65 -0.75)
+            (xy -0.15 0)
+            (xy -0.65 0.75)
+            (xy 0.5 0.75)
+          ) (width 0) (fill yes))
+      ))
+  )
   (footprint "Resistor_SMD:R_0603_1608Metric_Pad0.98x0.95mm_HandSolder" (layer "B.Cu")
     (at 131.455317 96.816534 180)
@@
   (via (at 138.46 104.78) (size 0.7) (drill 0.3) (layers "F.Cu" "B.Cu") (free) (net 10))
   (via (at 128.792838 103.794722) (size 0.7) (drill 0.3) (layers "F.Cu" "B.Cu") (free) (net 10))
+  (segment (start 130.552503 107.305677) (end 130.552503 106.457497) (width 0.25) (layer "B.Cu") (net 11))
+  (segment (start 130.552503 106.457497) (end 131.086202 105.923798) (width 0.25) (layer "B.Cu") (net 11))
+  (segment (start 131.086202 105.923798) (end 133.906645 105.923798) (width 0.25) (layer "B.Cu") (net 11))
+  (segment (start 133.906645 105.923798) (end 134.456647 105.373796) (width 0.25) (layer "B.Cu") (net 11))
   (segment (start 134.456647 105.373796) (end 134.456646 101.983015) (width 0.25) (layer "B.Cu") (net 11))
-  (segment (start 133.906645 105.923798) (end 134.456647 105.373796) (width 0.25) (layer "B.Cu") (net 11))
-  (segment (start 131.934385 105.923797) (end 133.906645 105.923798) (width 0.25) (layer "B.Cu") (net 11))
-  (segment (start 130.552503 107.305677) (end 131.934385 105.923797) (width 0.25) (layer "B.Cu") (net 11))
   (zone (net 6) (net_name "/Audio") (layer "F.Cu") (hatch edge 0.508)
     (priority 16962)
